File: Eagle/Omniboard.brd (EAGLE design)
At the start: 30 x 55 mm, 61 parts, among them IC1 AP2112K-3.3TRG1 3.3V, Q1 12MHz 3.2x2.5, Q2 BC817, Q3 BC817, Q4 MMBT2222A, SW1 ED_DPDT, U1 CH340T, U2 LMC7101AIM5, U3 MCP73213, U4 DRV8837, U5 DRV8837, U6 DRV8837, X1 ESP-12

Commit message: Changed to 1S lipo, button added, bugs fixed
Parts:
- removed SJ2: ID, SparkFun-Passives:PAD-JUMPER-2-NC_BY_PASTE_YES_SILK
- added C19, C21, C22, C23: 0.1uF, SparkFun-Capacitors:0402-CAP
- added C20: 4.7uF, SparkFun-Passives:0402-CAP
- added D2: BA340A, SparkFun-DiscreteSemi:SMA-DIODE
- added GND12, GND16: VIRTUAL_GND, alvaroferran:STARGND
- added JP7: M02POLAR_LOCK, SparkFun-Connectors:MOLEX-1X2_LOCK
- added L1: MPI4040R3-2R2-R, inductor-Eaton Bussmann:MPI4040R3-2R2-R
- added LED2: (no value), SparkFun-LED:LED-0603
- added R16: 330, SparkFun-Passives:0402-RES
- added U7: DRV8837, packages(ti):DSG
- C1: value 22pF -> 2.2uF; device SparkFun-Passives:0402-CAP -> SparkFun-Passives:0603-CAP
- C10: value 1uF -> 10uF 10V; device SparkFun-Passives:0603-CAP -> SparkFun-Passives:0402-CAP
- C11: value 10uF 10V -> 100nF; device SparkFun-Passives:0603-CAP -> SparkFun-Passives:0402-CAP
- C12, C16: value 0.1uF -> 10uF 10V; device SparkFun-Capacitors:0402-CAP -> SparkFun-Passives:0603-CAP
- C13: value 0.1uF -> 1uF; device SparkFun-Capacitors:0402-CAP -> SparkFun-Passives:0603-CAP
- C14: value 0.1uF -> 4.7uF; device SparkFun-Capacitors:0402-CAP -> SparkFun-Passives:0402-CAP
- C15: value 100nF -> 1uF; device SparkFun-Passives:0402-CAP -> SparkFun-Passives:0603-CAP
- C3: value 100nF -> 22pF
- C4: value 470pF -> 0.1uF; device SparkFun-Passives:0402-CAP -> SparkFun-Passives:0603-CAP
- C5: value 10uF 10V -> 100nF
- C6: value 100nF -> 470pF
- C7: value 10uF 10V -> 10nF
- C8: value 1uF -> 100pF
- C9: value 100nF -> 22uF; device SparkFun-Passives:0402-CAP -> SparkFun-Capacitors:0805
- D1: value BA340A -> B340A
- R10: value 1k -> 4.7k; device SparkFun-Passives:0402-RES -> resistor:R0402
- R11: value 1k -> 10k; device SparkFun-Passives:0402-RES -> resistor:R0402
- R12: value 330 -> 10k; device SparkFun-Passives:0402-RES -> resistor:R0402
- R14: value 2.32k -> 330
- R15: value 2.32k -> 2k
- R6: value 4.7k -> 620; device resistor:R0402 -> SparkFun-Passives:0603-RES
- R7: value 4.7k -> 30.9k; device resistor:R0402 -> SparkFun-Passives:0603-RES
- R8: device resistor:R0402 -> SparkFun-Passives:0603-RES
- R9: value 10k -> 4.7k
- SW1: value ED_DPDT -> RESET; device pighiXXX:ED_DPDT -> MySMD:157SW
- U1: value CH340T -> (none); device template:SSOP20 -> MIC2253_MLF12:MLF12_3.0MM_X_3.0MM
- U2: value LMC7101AIM5 -> CH340T; device linear:SOT23-5 -> template:SSOP20
- U3: value MCP73213 -> LMC7101AIM5; device alvaroferran:DFN10 -> linear:SOT23-5
- U4: value DRV8837 -> MCP73831; device packages(ti):DSG -> SparkFun-PowerIC:SOT23-5
- moved R10 36.5 mm to (4.06, 16.5), turned to 0 degrees
- moved R12 35.9 mm to (23.6, 11.4)
- moved C4 35.3 mm to (13.1, 42.5), flipped to the top
- moved R8 34.4 mm to (13.1, 43.8), turned to 180 degrees
- moved R11 33.5 mm to (20.3, 10.2), flipped to the top
- moved C12 33.4 mm to (24.8, 17.9), flipped to the bottom, turned to 180 degrees
- moved C16 33.1 mm to (28.3, 17.9), flipped to the bottom, turned to 0 degrees
- moved C1 31.6 mm to (13.1, 41.2)
- moved R6 30.2 mm to (17.4, 45.8), flipped to the top, turned to 180 degrees
- moved R7 29.8 mm to (17.4, 43.2), flipped to the top
- moved C7 29.6 mm to (13.1, 45.1), flipped to the top, turned to 0 degrees
- moved C17 24.3 mm to (7.62, 47.2), turned to 90 degrees
- moved C15 24.2 mm to (28.3, 24.5), flipped to the bottom, turned to 180 degrees
- moved C6 21.3 mm to (4.06, 8.38), flipped to the bottom, turned to 0 degrees
- moved U5 21.3 mm to (9.91, 47.5), turned to 270 degrees
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Connections:
- new net AGND: C4.1, C7.1, GND16.P$1, R8.2, U1.4
- new net N$16: R6.1, U1.12
- new net N$24: C8.1, R7.1, R8.1, U1.3
- new net N$3: C7.2, R6.2
- new net N$4: C4.2, U1.2
- new net PGND: C1.1, C9.1, GND12.P$1, U1.5, U1.6
- new net VDD: C21.1, C22.1, C23.1, C8.2, C9.2, D1.C, R7.2, U1.9, U3.2, U5.1, U6.1, U7.1
- net 3.3V: now also C15.2, C16.1, C17.1, C18.1, C19.1, LED2.A, U2.19, U2.5, U3.3, U7.7, U7.8; no longer C12.1, C13.1, C14.1, C3.2, C6.1, U1.19, U1.5, U2.4, U4.7, U4.8
- net D+: now also U2.6; no longer U1.6
- net D-: now also U2.7; no longer U1.7
- net GND: now also C13.1, C15.1, C19.2, C20.2, C21.2, C22.2, C23.2, GND12.P$2, GND16.P$2, R16.1, SW1.2, U2.8, U3.5, U4.2, U7.4, U7.PAD; no longer C1.1, C13.2, C15.2, C4.2, C7.2, C8.1, C9.2, R11.2, R14.2, U1.8, U2.5, U3.8, U3.9, U4.4, U4.PAD
- net GPIO0: now also SW1.1, U7.6; no longer U6.6
- net GPIO13: now also U5.6; no longer U4.6
- net GPIO15: now also U5.5; no longer U4.5
- net GPIO2: now also U7.5; no longer U6.5
- net GPIO4: now also U6.6; no longer U5.6
- net GPIO5: now also U6.5; no longer U5.5
- net MOT1A: now also U6.2; no longer U5.2
- net MOT1B: now also U6.3; no longer U5.3
- net MOT2A: now also U7.2; no longer U6.2
- net MOT2B: now also U7.3; no longer U6.3
- net MOT3A: now also U5.2; no longer U4.2
- net MOT3B: now also U5.3; no longer U4.3
- net N$1: now also R10.2, R9.2; no longer R6.2, R7.2
- net N$10: now also R11.2, U2.16; no longer R8.2, U1.16
- net N$11: now also R15.1, U4.5; no longer R14.1, SJ2.2, U3.10
- net N$12: now also D1.A, L1.P$2, U1.7, U1.8; no longer R15.1, SJ2.1
- net N$13: now also R14.1, U4.1; no longer R12.1, U3.7
- net N$15: now also LED2.C, R16.2; no longer R10.2, R11.1, U2.3
- net N$17: now also U3.1; no longer U2.1
- net N$2: now also R12.2, U2.15; no longer R9.2, U1.15
- net N$5: now also R14.2; no longer R12.2
- net N$6: now also R11.1; no longer R8.1
- net N$7: now also R12.1; no longer R9.1
- net RESET: now also C6.1; no longer C4.1
- net RXD: now also U2.3; no longer U1.3
- net SCL: now also R10.1; no longer R7.1
- net SDA: now also R9.1; no longer R6.1
- net TXD: now also U2.4; no longer U1.4
- net VBAT: now also JP7.2; no longer SW1.1, SW1.4
- net VIN: now also C12.1, C13.2, C14.1, D2.C, U4.4; no longer C7.1, C8.2, C9.1, D1.C, U3.1, U3.2
- net V_BATT: now also C1.2, C20.1, D2.A, JP7.1, L1.P$1, U1.10, U1.11, U4.3; no longer C15.1, C16.1, C17.1, C18.1, D1.A, R10.1, SW1.2, SW1.5, U2.2, U3.3, U4.1, U5.1, U6.1
- net XI: now also C2.2, U2.9; no longer C1.2, U1.9
- net XO: now also C3.2, U2.10; no longer C2.2, U1.10
Routing:
- net VDD: track 0.00 -> 93.1 mm, vias 0 -> 9
- net V_BATT: track 99.9 -> 67.8 mm, vias 8 -> 6
- net VBAT: track 21.7 -> 7.38 mm
- net N$12: track 1.21 -> 13.9 mm, vias 0 -> 2
- net AGND: track 0.00 -> 9.73 mm, vias 0 -> 2
- net 3.3V: track 146.4 -> 155.0 mm, vias 14 -> 15
- net N$24: track 0.00 -> 8.68 mm
- net VIN: track 75.9 -> 69.2 mm, vias 1 -> 3
- net PGND: track 0.00 -> 5.75 mm
- net N$16: track 0.00 -> 5.09 mm
- net N$4: track 0.00 -> 3.68 mm, vias 0 -> 2
- net N$11: track 4.89 -> 1.29 mm, vias 1 -> 0
- net GPIO0: track 44.4 -> 47.9 mm
- net N$3: track 0.00 -> 3.11 mm
- net N$15: track 2.92 -> 0.89 mm
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Other:
- board text added: "PROG"
- board text added: "PWR"
- board text added: "SWITCH"
- board text removed: "FAST CHARGE"
- board text removed: "ON / OFF"

Commit message: Project updated
Parts:
- C10: value 10uF 10V -> 22pF
- C11: value 100nF -> 22pF
- C12: value 10uF 10V -> 1uF
- C13: value 1uF -> 100nF; device SparkFun-Passives:0603-CAP -> SparkFun-Passives:0402-CAP
- C17: value 0.1uF -> 4.7uF; device SparkFun-Capacitors:0402-CAP -> SparkFun-Passives:0402-CAP
- C2: value 22pF -> 0.1uF; device SparkFun-Passives:0402-CAP -> SparkFun-Passives:0603-CAP
- C20: value 4.7uF -> 0.1uF; device SparkFun-Passives:0402-CAP -> SparkFun-Capacitors:0402-CAP
- C3: value 22pF -> 470pF
- C4: value 0.1uF -> 10nF
- C5: value 100nF -> 100pF; device SparkFun-Passives:0402-CAP -> SparkFun-Passives:0603-CAP
- C6: value 470pF -> 22uF; device SparkFun-Passives:0402-CAP -> SparkFun-Capacitors:0805
- C7: value 10nF -> 10uF 10V; device SparkFun-Passives:0603-CAP -> SparkFun-Passives:0402-CAP
- C8: value 100pF -> 100nF; device SparkFun-Passives:0603-CAP -> SparkFun-Passives:0402-CAP
- C9: value 22uF -> 10uF 10V; device SparkFun-Capacitors:0805 -> SparkFun-Passives:0603-CAP
- JP1: value M02POLAR_LOCK -> USB_MICROB; device SparkFun-Connectors:MOLEX-1X2_LOCK -> SparkFun-Connectors:USB-B-MICRO-SMD_V03
- JP2: value USB_MICROB_PLUGCONN-11752 -> M02POLAR_LOCK; device SparkFun-Connectors:USB-B-MICRO-SMD_V03 -> SparkFun-Connectors:MOLEX-1X2_LOCK
- JP3: value M02POLAR_LOCK -> (none); device SparkFun-Connectors:MOLEX-1X2_LOCK -> SparkFun-Connectors:1X05_LOCK
- JP4: value M02POLAR_LOCK -> M02LOCK; device SparkFun-Connectors:MOLEX-1X2_LOCK -> SparkFun-Connectors:1X02_LOCK
- JP5: value (none) -> M02POLAR_LOCK; device SparkFun-Connectors:1X05_LOCK -> SparkFun-Connectors:MOLEX-1X2_LOCK
- JP6: value M02LOCK -> M02POLAR_LOCK; device SparkFun-Connectors:1X02_LOCK -> SparkFun-Connectors:MOLEX-1X2_LOCK
- Q2: value BC817 -> MMBT2222A; device transistor-npn:SOT23-BEC -> SparkFun-DiscreteSemi:SOT23-3
- Q4: value MMBT2222A -> BC817; device SparkFun-DiscreteSemi:SOT23-3 -> transistor-npn:SOT23-BEC
- R11: value 10k -> 330; device resistor:R0402 -> SparkFun-Passives:0402-RES
- R12: value 10k -> 10K; device resistor:R0402 -> SparkFun:0402-RES
- R13: value 10K -> 10k; device SparkFun:0402-RES -> resistor:R0402
- R14: value 330 -> 10k; device SparkFun-Passives:0402-RES -> resistor:R0402
- R15: value 2k -> 330
- R16: value 330 -> 2k
- U2: value CH340T -> LMC7101AIM5; device template:SSOP20 -> linear:SOT23-5
- U3: value LMC7101AIM5 -> CH340T; device linear:SOT23-5 -> template:SSOP20
- moved JP2 50.1 mm to (22.9, 52.1), turned to 180 degrees
- moved C2 32.8 mm to (13.1, 42.5), turned to 0 degrees
- moved R13 32.5 mm to (20.3, 10.2), flipped to the top, turned to 0 degrees
- moved C6 32.5 mm to (13.1, 39.6), flipped to the top, turned to 180 degrees
- moved R12 31.3 mm to (21.3, 42.7), flipped to the bottom, turned to 270 degrees
- moved Q4 31.0 mm to (23.6, 8.89), flipped to the top
- moved R11 27.8 mm to (15.0, 37.5)
- moved R14 27.4 mm to (23.6, 11.4), turned to 180 degrees
- moved JP1 27.1 mm to (24.1, 2.03)
- moved Q2 27.0 mm to (22.2, 39.9), flipped to the bottom, turned to 180 degrees
- moved JP5 26.3 mm to (27.2, 29.0)
- moved C3 25.7 mm to (4.06, 8.38), flipped to the bottom
- moved C5 25.3 mm to (17.4, 44.5), turned to 0 degrees
- moved C9 24.7 mm to (24.8, 17.9), flipped to the bottom
- moved C21 22.0 mm to (22.4, 27.9), turned to 180 degrees
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- renumbered GND12 to GND10, GND16 to GND13
Connections:
- net 3.3V: now also C13.2, C20.1, C7.2, C8.1, JP3.5, U2.3, U3.19, U3.5; no longer C10.2, C11.1, C17.1, C5.2, JP5.5, U2.19, U2.5, U3.3
- net ADC: now also JP3.1; no longer JP5.1
- net AGND: now also C2.1; no longer C7.1
- net D+: now also JP1.D+1, U3.6; no longer JP2.D+1, U2.6
- net D-: now also JP1.D-1, U3.7; no longer JP2.D-1, U2.7
- net GND: now also C11.1, C12.1, C3.2, C7.1, C8.2, C9.2, JP1.GND1, JP1.SHIELD1, JP1.SHIELD2, JP1.SHIELD3, JP3.2, JP4.2, Q2.2, R15.1, R16.2, U2.5, U3.8; no longer C11.2, C12.2, C2.1, C3.1, C5.1, C6.2, JP2.GND1, JP2.SHIELD1, JP2.SHIELD2, JP2.SHIELD3, JP5.2, JP6.2, Q4.2, R15.2, R16.1, U2.8, U3.5
- net GPIO0: now also Q3.C, U6.6; no longer Q2.C, U7.6
- net GPIO13: now also U7.6; no longer U5.6
- net GPIO15: now also U7.5; no longer U5.5
- net GPIO2: now also U6.5; no longer U7.5
- net GPIO4: now also U5.6; no longer U6.6
- net GPIO5: now also U5.5; no longer U6.5
- net MOT1A: now also JP5.1, U5.2; no longer JP1.1, U6.2
- net MOT1B: now also JP5.2, U5.3; no longer JP1.2, U6.3
- net MOT2A: now also JP6.1, U6.2; no longer JP3.1, U7.2
- net MOT2B: now also JP6.2, U6.3; no longer JP3.2, U7.3
- net MOT3A: now also JP7.1, U7.2; no longer JP4.1, U5.2
- net MOT3B: now also JP7.2, U7.3; no longer JP4.2, U5.3
- net N$10: now also Q4.E, R13.2, U3.16; no longer Q3.E, R11.2, U2.16
- net N$11: now also R16.1; no longer R15.1
- net N$13: now also R11.1; no longer R14.1
- net N$14: now also JP1.VBUS1; no longer JP2.VBUS1
- net N$15: now also R15.2; no longer R16.2
- net N$17: now also R12.1, U2.1; no longer R13.1, U3.1
- net N$2: now also Q3.E, R14.2, U3.15; no longer Q2.E, R12.2, U2.15
- net N$24: now also C5.1; no longer C8.1
- net N$3: now also C4.2; no longer C7.2
- net N$4: now also C2.2; no longer C4.2
- net N$5: now also R11.2; no longer R14.2
- net N$6: now also Q3.B, R13.1; no longer Q2.B, R11.1
- net N$7: now also Q4.B, R14.1; no longer Q3.B, R12.1
- net N$8: now also Q2.1, R12.2; no longer Q4.1, R13.2
- net N$9: now also Q2.3; no longer Q4.3
- net PGND: now also C6.1; no longer C9.1
- net RESET: now also C3.1, Q4.C; no longer C6.1, Q3.C
- net RXD: now also U3.3; no longer U2.3
- net SCL: now also JP3.3; no longer JP5.3
- net SDA: now also JP3.4; no longer JP5.4
- net TXD: now also U3.4; no longer U2.4
- net VBAT: now also JP2.2, JP4.1; no longer JP6.1, JP7.2
- net VDD: now also C5.2, C6.2, U2.2; no longer C8.2, C9.2, U3.2
- net VIN: now also C12.2, C9.1; no longer C12.1, C13.2
- net V_BATT: now also C17.1, JP2.1, U2.4; no longer C20.1, JP7.1, U3.4
- net XI: now also C10.2, U3.9; no longer C2.2, U2.9
- net XO: now also C11.2, U3.10; no longer C3.2, U2.10
Other:
- board text added: "L1"
